Commit message: Working Gazebo

File: install/rarm/share/rarm/urdf/GP7.urdf.xacro (robot description, xacro)
@@ -1,4 +1,6 @@
 <?xml version="1.0"?>
 <robot xmlns:xacro="http://www.ros.org/wiki/xacro">
+    <xacro:property name="joint_damping" value="5.0"/>
+  <xacro:property name="joint_friction" value="0.3"/>
    <link name="world"/>
   <joint
@@ -12,5 +14,5 @@
     <child
       link="base_link" />
-      <dynamics damping="2.0" friction="1.0"/>
+       <dynamics damping="${joint_damping}" friction="${joint_friction}"/>
   </joint>
 <link
@@ -111,4 +113,5 @@
       effort="30"
       velocity="6.545" />
+       <dynamics damping="${joint_damping}" friction="${joint_friction}"/>
   </joint>
   <link
@@ -165,8 +168,9 @@
       xyz="0 0 -1" />
     <limit
-      lower="-1.135"
-      upper="2.53"
+      lower="-2.53"
+      upper="1.135"
       effort="30"
       velocity="5.497" />
+        <dynamics damping="${joint_damping}" friction="${joint_friction}"/>
   </joint>
   <link
@@ -227,4 +231,5 @@
       effort="30"
       velocity="7.155" />
+       <dynamics damping="${joint_damping}" friction="${joint_friction}"/>
   </joint>
   <link
@@ -285,4 +290,5 @@
       effort="30"
       velocity="9.599" />
+       <dynamics damping="${joint_damping}" friction="${joint_friction}"/>
   </joint>
   <link
@@ -343,4 +349,5 @@
       effort="30"
       velocity="9.599" />
+       <dynamics damping="${joint_damping}" friction="${joint_friction}"/>
   </joint>
   <link
@@ -401,4 +408,5 @@
       effort="30"
       velocity="17.453" />
+       <dynamics damping="${joint_damping}" friction="${joint_friction}"/>
   </joint>
   <link
@@ -459,4 +467,5 @@
       effort="30"
       velocity="10" />
+       <dynamics damping="${joint_damping}" friction="${joint_friction}"/>
   </joint>
   <link
@@ -513,8 +522,10 @@
       xyz="0 0 1" />
     <limit
-      lower="0"
-      upper="1.57"
+      lower="-1.57"
+      upper="0"
       effort="30"
       velocity="10" />
+      <mimic joint="J7" multiplier="1.0" offset="0"/>
+       <dynamics damping="${joint_damping}" friction="${joint_friction}"/>
   </joint>
   </robot>

File: install/rarm/share/rarm/urdf/GP7_ros2_control.urdf.xacro (robot description, xacro)
@@ -17,6 +17,6 @@
             <joint name="J2">
                 <command_interface name="position">
-                    <param name="min">-1.135</param>
-                    <param name="max">2.53</param>
+                    <param name="min">-2.53</param>
+                    <param name="max">1.135</param>
                 </command_interface>
                 <state_interface name="position"/>
@@ -59,4 +59,10 @@
             </joint>
             <joint name="J8">
+                <param name="mimic">J7</param>
+                <param name="multiplier">1.0</param>
+                <state_interface name="position"/>
+                <state_interface name="velocity"/>
+            </joint>
+            <!-- <joint name="J8">
                 <command_interface name="position">
                     <param name="min">0</param>
@@ -65,5 +71,5 @@
                 <state_interface name="position"/>
                 <state_interface name="velocity"/>
-            </joint>
+            </joint>-->
             <!-- <joint name="${prefix}gripper_controller">
                 <command_interface name="position">
